File: besc g2 io.sch (KiCad schematic (older format))
At the start: 34 parts, among them J10 614105150721, J11 THROTTLE, J12 MOTOR SENSOR, J13 THROTTLE 2 (BRAKE), J14 SERIAL, J15 IGNITION, J16 CAN, J8 SWD, J9 RC PWM, U10 TJA1051T-3, U9 USBLC6-2SC6

Commit message: Added brakes, i2c
Signed-off-by: manianac <manianac@gmail.com>
Parts:
- removed J10: 614105150721, Connector_USB:USB_Micro-B_Wuerth_614105150721_Vertical_CircularHoles, symbol Connector:USB_B_Micro
- added C63: 100n, Capacitor_SMD:C_0603_1608Metric, symbol Device:C_Small
- added J10: USB_C_Receptacle_USB2.0, BESC-G2:GCT_USB4120-03-C_REVA, symbol Connector:USB_C_Receptacle_USB2.0
- added J18: BRAKE_SW, Connector_PinHeader_2.54mm:PinHeader_1x02_P2.54mm_Vertical, symbol Connector_Generic:Conn_01x02
- added J19: REVERSE_SW, Connector_PinHeader_2.54mm:PinHeader_1x02_P2.54mm_Vertical, symbol Connector_Generic:Conn_01x02
- added J20: I2C, Connector_PinSocket_2.54mm:PinSocket_1x04_P2.54mm_Vertical, symbol Connector_Generic:Conn_01x04
- added R100, R65: 5K1, Resistor_SMD:R_0603_1608Metric, symbol Device:R_Small
- added R101, R103: 1k8, Resistor_SMD:R_0603_1608Metric, symbol Device:R_Small
- added R102, R104: 3k3, Resistor_SMD:R_0603_1608Metric, symbol Device:R_Small
- added U7: LMV358, Package_SO:SOIC-8_3.9x4.9mm_P1.27mm, symbol Amplifier_Operational:LMV358
- J14: footprint Connector_PinHeader_2.54mm:PinHeader_1x05_P2.54mm_Vertical -> Connector_PinHeader_2.54mm:PinHeader_1x04_P2.54mm_Vertical; symbol Connector_Generic:Conn_01x05 -> Connector_Generic:Conn_01x04
- J9: value RC PWM -> PAS
- U9: symbol Power_Protection:USBLC6-2SC6 -> besc-g2-rescue:USBLC6-2SC6-Power_Protection
Connections:
- net labels added: BRAKE_SW, I2C_SCL, I2C_SDA, PAS_ADC, REVERSE_SW, UART_RX, UART_TX
- net labels removed: RC_PWM, RX, TX
- wire segments 143 -> 185
- no-connect marks 0 -> 2
Other:
- note added: "We let the STM32 pull this up\nso that we can redefine this if need be"
- moved on the sheet: C85, C86, C87, C88, J11, J12, J13, R74, R76, R77, R78, R79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
